File: PCB/IDC_adapter.kicad_pcb (KiCad board)
At the start: 2 copper layers, 44.5 x 44.5 mm, 4 parts, among them J1 Portal_Jack, J2 Panel_Jack

Commit message: update pcb design
Parts:
- added REF**: MountingHole_2.5mm, MountingHole:MountingHole_2.5mm, F.Cu at (132.7, 104.8)
- J2: moved to F.Cu
- moved J2 17.8 mm to (165.1, 113.7)
- moved J1 3.81 mm to (152.4, 95.9)
Routing:
- net Net-(J1-Pin_2): track 12.7 -> 48.1 mm
- net Net-(J1-Pin_4): track 12.7 -> 47.4 mm
- net Net-(J1-Pin_6): track 12.7 -> 46.2 mm
- net Net-(J1-Pin_8): track 12.7 -> 45.0 mm
- net Net-(J1-Pin_10): track 12.7 -> 43.2 mm
- net Net-(J1-Pin_12): track 12.7 -> 41.7 mm
- net Net-(J1-Pin_14): track 12.7 -> 40.2 mm
- net Net-(J1-Pin_1): track 18.8 -> 46.2 mm
- net Net-(J1-Pin_3): track 18.8 -> 44.2 mm
- net Net-(J1-Pin_5): track 18.8 -> 42.8 mm
- net Net-(J1-Pin_7): track 18.8 -> 41.4 mm
- net Net-(J1-Pin_9): track 18.8 -> 39.8 mm
- net Net-(J1-Pin_11): track 18.8 -> 38.1 mm
- net Net-(J1-Pin_13): track 18.8 -> 36.0 mm
- net Net-(J1-Pin_15): track 18.9 -> 30.5 mm
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Other:
- board text added: "1.75in x 1.75in M2.5 hole"
- board text added: "2023-08-23 1.0.0"
- board text removed: "1.75in x 1.75in M2.5 holes"
- board text removed: "2023-08-17 0.0.0"
